File: hardware/hardgfx-black/hardgfx-black.kicad_sch (KiCad schematic)
At the start: 16 parts, among them SW1 SW_MEC_5E, U1 STM32H745BITx, X1 25MHz, Y1 ECS-.327-6-34R-TR

Commit message: Schematic with the LCD and FLASH memory connection to the MCU ready.
Parts:
- added R107, R108, R109, R110, R111, R112, R113, R114, R115, R116: 33, symbol Device:R
Connections:
- net LCD_MODE: now reaches U1.130 (PG2)
- net FMC_BA0: now reaches U1.134 (PG4)
- net FMC_BA1: now reaches U1.135 (PG5)
- net LCD_DCLK: now reaches U1.137 (PG7)
- net at U1.180 (PG9): now also R115.1
- net LCD_B2: now reaches U1.181 (PG10)
- net LCD_B4: now reaches U1.183 (PG12)
- net at U1.185 (PG14): now also R116.1
- net FMC_A0: now reaches U1.22 (PF0)
- net FMC_A1: now reaches U1.23 (PF1)
- net FMC_A2: now reaches U1.24 (PF2)
- net FMC_A3: now reaches U1.25 (PF3)
- net FMC_A4: now reaches U1.26 (PF4)
- net FMC_A5: now reaches U1.27 (PF5)
- net LCD_B0: now reaches U1.3 (PE4)
- net at U1.30 (PF6): now also R112.2
- net at U1.31 (PF7): now also R111.2
- net at U1.32 (PF8): now also R109.2
- net at U1.33 (PF9): now also R110.2
- net LCD_DE: now reaches U1.34 (PF10)
- net at U1.48 (PH2): now also R113.1
- net at U1.51 (PH3): now also R114.1
- net FMC_A6: now reaches U1.68 (PF12)
- net FMC_A7: now reaches U1.69 (PF13)
- net FMC_A8: now reaches U1.70 (PF14)
- net FMC_A9: now reaches U1.71 (PF15)
- net FMC_A10: now reaches U1.72 (PG0)
- net FMC_A11: now reaches U1.75 (PG1)
- net FMC_D4: now reaches U1.76 (PE7)
- net FMC_D5: now reaches U1.77 (PE8)
- net FMC_D6: now reaches U1.78 (PE9)
- net FMC_D7: now reaches U1.81 (PE10)
- net FMC_D8: now reaches U1.82 (PE11)
- net FMC_D9: now reaches U1.83 (PE12)
- net FMC_D10: now reaches U1.84 (PE13)
- net FMC_D11: now reaches U1.85 (PE14)
- net FMC_D12: now reaches U1.86 (PE15)
- net FMC_D16: now reaches U1.94 (PH8)
- net FMC_D17: now reaches U1.95 (PH9)
- net ~{LCD_RST}: now reaches U1.101 (PB12)
- net LCD_UD: now reaches U1.102 (PB13)
- net LCD_LR: now reaches U1.103 (PB14)
- net ~{LCD_WAKE}: now reaches U1.104 (PB15)
- net FMC_D13: now reaches U1.105 (PD8)
- net FMC_D14: now reaches U1.106 (PD9)
- net FMC_D15: now reaches U1.107 (PD10)
- net ~{LCD_INT}: now reaches U1.110 (PD11)
- net LCD_SCL: now reaches U1.111 (PD12)
- net LCD_SDA: now reaches U1.112 (PD13)
- net FMC_D0: now reaches U1.115 (PD14)
- net FMC_D1: now reaches U1.116 (PD15)
- net LCD_HSYNC: now reaches U1.142 (PC6)
- net LCD_B3: now reaches U1.146 (PA8)
- net LCD_B1: now reaches U1.148 (PA10)
- net FMC_D2: now reaches U1.170 (PD0)
- net FMC_D3: now reaches U1.171 (PD1)
- net LCD_B6: now reaches U1.195 (PB8)
- net LCD_B7: now reaches U1.196 (PB9)
- net LCD_R5: now reaches U1.38 (PC0)
- net LCD_R2: now reaches U1.46 (PA1)
- net LCD_R1: now reaches U1.47 (PA2)
- net LCD_B5: now reaches U1.54 (PA3)
- net LCD_VSYNC: now reaches U1.57 (PA4)
- net LCD_R4: now reaches U1.58 (PA5)
- net LCD_BCKL: now reaches U1.59 (PA6)
- net LCD_R3: now reaches U1.63 (PB0)
- net LCD_R6: now reaches U1.64 (PB1)
- net at U1.65 (PB2): now also R107.2
- net at U1.87 (PB10): now also R108.2
- net LCD_DITH: now reaches U1.88 (PB11)
- net LCD_R7: now reaches U1.117 (PJ6)
- net LCD_G0: now reaches U1.118 (PJ7)
- net LCD_G1: now reaches U1.121 (PJ8)
- net LCD_G2: now reaches U1.122 (PJ9)
- net LCD_G3: now reaches U1.123 (PJ10)
- net LCD_G4: now reaches U1.124 (PJ11)
- net LCD_G5: now reaches U1.127 (PK0)
- net LCD_G6: now reaches U1.128 (PK1)
- net LCD_G7: now reaches U1.129 (PK2)
- net LCD_R0: now reaches U1.66 (PI15)
- new net QSPI_BK1_IO0: R109.1
- new net QSPI_BK1_IO1: R110.1
- new net QSPI_BK1_IO2: R111.1
- new net QSPI_BK1_IO3: R112.1
- new net QSPI_BK1_NCS: R108.1
- new net QSPI_BK2_IO0: R113.2
- new net QSPI_BK2_IO1: R114.2
- new net QSPI_BK2_IO2: R115.2
- new net QSPI_BK2_IO3: R116.2
- new net QSPI_CLK: R107.1
Other:
- moved on the sheet: TP1
