File: hardware/hardgfx-black/hardgfx-black.kicad_sch (KiCad schematic)
At the start: 30 parts, among them J28 Conn_01x08, J29 Conn_01x08, J30 Conn_01x08, J31 Conn_01x08, SW1 SW_MEC_5E, U1 STM32H745BITx, X1 25MHz, Y1 ECS-.327-6-34R-TR

Commit message: Adding application note PDF document and change backlight controller.
Parts:
- J28, J29, J30, J31: mouser# 200-TSW10807GS -> 200-TSW10407GS
Changed lines of the file:
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@@
       (effects (font (size 1.27 1.27)) hide)
     )
-    (property "mouser#" "200-TSW10807GS" (id 7) (at 345.44 229.87 0)
+    (property "mouser#" "200-TSW10407GS" (id 7) (at 345.44 229.87 0)
       (effects (font (size 1.27 1.27)) hide)
     )
@@
       (effects (font (size 1.27 1.27)) hide)
     )
-    (property "mouser#" "200-TSW10807GS" (id 7) (at 302.26 229.87 0)
+    (property "mouser#" "200-TSW10407GS" (id 7) (at 302.26 229.87 0)
       (effects (font (size 1.27 1.27)) hide)
     )
@@
       (effects (font (size 1.27 1.27)) hide)
     )
-    (property "mouser#" "200-TSW10807GS" (id 7) (at 302.26 182.88 0)
+    (property "mouser#" "200-TSW10407GS" (id 7) (at 302.26 182.88 0)
       (effects (font (size 1.27 1.27)) hide)
     )
@@
       (effects (font (size 1.27 1.27)) hide)
     )
-    (property "mouser#" "200-TSW10807GS" (id 7) (at 345.44 182.88 0)
+    (property "mouser#" "200-TSW10407GS" (id 7) (at 345.44 182.88 0)
       (effects (font (size 1.27 1.27)) hide)
     )
@@
     )
     (path "/703bab7f-0bb8-4b10-89a6-009fe08e4f5b/79f2c0a1-c6b8-4582-8f8a-407f8250d0c2"
-      (reference "J21") (unit 1) (value "Conn_ARM_JTAG_SWD_20") (footprint "Connector_PinHeader_2.54mm:PinHeader_2x10_P2.54mm_Vertical_SMD")
+      (reference "J21") (unit 1) (value "Conn_ARM_JTAG_SWD_20") (footprint "Connector_IDC:IDC-Header_2x10_P2.54mm_Latch6.5mm_Vertical")
     )
     (path "/58af4faa-dce1-4105-a7e2-ce501536c4bc/95530a8d-3ffb-464e-bc5a-b002cfa205ef"
@@
       (reference "U7") (unit 1) (value "IS42S32800J-6TLI") (footprint "IS42S32800J-6TLI:SOP50P1176X120-86N")
     )
-    (path "/7e86bd46-cd49-4013-a820-6e307d2e7505/9bc74719-29e6-4a54-b90d-9d67aa557a3c"
-      (reference "U8") (unit 1) (value "TPS61041DRVT") (footprint "Package_SON:WSON-6-1EP_2x2mm_P0.65mm_EP1x1.6mm")
+    (path "/7e86bd46-cd49-4013-a820-6e307d2e7505/47758ecf-2409-4bc7-8924-a639dd60d1c9"
+      (reference "U8") (unit 1) (value "TPS61041DBV") (footprint "Package_TO_SOT_SMD:SOT-23-5")
     )
     (path "/58af4faa-dce1-4105-a7e2-ce501536c4bc/46e3df63-50fc-48a7-9c2b-0b105fdb891a"
@@
     )
     (path "/58af4faa-dce1-4105-a7e2-ce501536c4bc/6d4da7fb-68f8-459d-815a-386dfd8063f8"
-      (reference "U10") (unit 1) (value "USBLC6-4SC6") (footprint "Package_TO_SOT_SMD:SOT-23-6")
+      (reference "U10") (unit 1) (value "USBLC6-4SC6Y") (footprint "Package_TO_SOT_SMD:SOT-23-6_Handsoldering")
     )
     (path "/58af4faa-dce1-4105-a7e2-ce501536c4bc/3f32ec1a-c27b-437c-9093-91068bc4c580"
