File: hardware/hardgfx-black/hardgfx-black.kicad_pcb (KiCad board)
At the start: 2 copper layers, 7.5 x 2 mm, 250 parts, among them J1 Input Voltage, J10 Conn_01x02, J11 Conn_01x02, J12 FH12-50S-0.5SH, J13 FH12-10S-0.5SH, J14 ~{LCD_RST}, J15 ~{LCD_WAKE}, J16 MODE, J17 LR, J18 UD, J19 DITH, J2 Conn_01x02, J20 Micro_SD_Card_Det, J21 Conn_ARM_JTAG_SWD_20, J22 USB_OTG, J23 WIFI_GPIO, J24 WIFI_GPIO, J25 Boot option, J26 WIFI_UART, J27 JTAG, J28 Conn_01x08, J29 Conn_01x08, J3 Conn_01x02, J30 Conn_01x08, J31 Conn_01x08, J4 Conn_01x02, J5 Conn_01x02, J6 Conn_01x02, J7 Conn_01x02, J8 Conn_01x02, J9 Conn_01x02, Q1 BSR14, SW1 SW_MEC_5E, SW2 SW_MEC_5E, SW3 WIFI_UART, U1 STM32H745BITx, U10 USBLC6-4SC6, U11 ESP32-WROOM-32, U2 MIC4575-5.0WU, U3 ST1L05APU33R, U4 LD1117S18TR, U5 MT25QL512ABB8ESF-0AAT, U6 MT25QL512ABB8ESF-0AAT, U7 IS42S32800J-6TLI, U8 TPS61041DRVT, U9 STMPS2151MTR, X1 25MHz, Y1 ECS-.327-6-34R-TR

Commit message: Adding application note PDF document and change backlight controller.
Parts:
- J21: footprint Connector_PinHeader_2.54mm:PinHeader_2x10_P2.54mm_Vertical_SMD -> Connector_IDC:IDC-Header_2x10_P2.54mm_Latch6.5mm_Vertical
- U8: value TPS61041DRVT -> TPS61041DBV; footprint Package_SON:WSON-6-1EP_2x2mm_P0.65mm_EP1x1.6mm -> Package_TO_SOT_SMD:SOT-23-5
- moved R9 233.0 mm to (99.1, 150.4)
- moved C42 229.5 mm to (99.1, 144.3), turned to 180 degrees
- moved R7 226.1 mm to (99.1, 147.3), turned to 180 degrees
- moved R8 222.6 mm to (99.1, 141.2)
- moved C43 213.8 mm to (99.1, 131.1), turned to 180 degrees
- moved R13 212.1 mm to (99.1, 136.7)
- moved R15 208.7 mm to (116.3, 136.7)
- moved R12 206.2 mm to (99.1, 127.5)
- moved U5 204.8 mm to (107.7, 145.8)
- moved U6 203.1 mm to (107.7, 132.1)
- moved R11 197.6 mm to (116.3, 150.4)
- moved CR3 197.0 mm to (307.3, 111.3)
- moved CR2 196.9 mm to (307.3, 106.2)
- moved R14 195.4 mm to (116.3, 129.0)
- moved C15 190.8 mm to (277.1, 62.8)
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Connections:
- J12 pad 3: Net-(R81-Pad1) -> Net-(J12-Pad3)
- J12 pad 4: Net-(R81-Pad1) -> Net-(J12-Pad3)
- R81 pad 1: Net-(R81-Pad1) -> Net-(J12-Pad3)
- U8 pad 1: GNDD -> Net-(D2-Pad2)
- U8 pad 2: +5V -> GNDD
- U8 pad 3: /LCD_BCKL -> Net-(J12-Pad3)
- U8 pad 4: Net-(R81-Pad1) -> /LCD_BCKL
- U8 pad 5: unconnected-(U8-Pad5) -> +5V
Other:
- outline, holes or cut-outs redrawn
