File: hardware/hardgfx-black/hardgfx-black_sdram.kicad_sch (KiCad schematic)
At the start: 70 parts, among them U7 IS42S32800J-6TLI

Commit message: Added generic SDRAM configuration using macros.
Other:
- note added: "* Reference the plane using GND or PWR (if PWR, add 10nf stitching cap between PWR and GND * Trace the impedance: 50 Ω ± 10% to 110MHz * The maximum trace length should be below 120mm. If the signal trace exceeds this trace-length/speed criterion, then a termination should be used. * Match the trace lengths for the data group within ± 10 mm of each other to diminish the skew. * Placing the clock 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"
- note removed: "* Reference the plane using GND or PWR (if PWR, add 10nf stitching cap between PWR and GND * Trace the impedance: 50 Ω ± 10% * The maximum trace length should be below 120mm. If the signal trace exceeds this trace-length/speed criterion, then a termination should be used. * Match the trace lengths for the data group within ± 10 mm of each other to diminish the skew. * Placing the clock (SDCLK) si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"
- moved on the sheet: C44, C45, C46, C47, C48, C49, C50, C51, C52, C53, C54, C55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
